File: Circuit Design/Circuit Design.kicad_sch (KiCad schematic)
At the start: 31 parts, among them J1 Power Header, J2 Scale Header, J3 Flowmeter Header, J4 IR Header, J6 Keypad Headers, Q1 2N3905, SW1 SW_MEC_5G, SW2 SW_MEC_5G, SW3 SW_MEC_5G, U1 HX711, U2 74LVC3G14

Commit message: Power Sche
Parts:
- renumbered C4 to C1, C5 to C2, C6 to C3, C7 to C4, C2 to C5, C1 to C6, C3 to C7, D2 to D1, D3 to D2, D1 to D3, J6 to J3, J3 to J5, R8 to R1, R1 to R10, R9 to R2, R10 to R3, R6 to R4, R7 to R5, R5 to R6, R3 to R7, R4 to R8, R2 to R9, U2 to U1, U1 to U2

Commit message: Adding MCU blank sheet and
Parts:
- removed J1: Power Header, Connector_Molex:Molex_KK-396_A-41791-0002_1x02_P3.96mm_Vertical, symbol Connector:Conn_01x02_Male
Other:
- added sheet MCU (MCU.kicad_sch)
Changed lines of the file:
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@@
-    (stroke (width 0) (type default) (color 0 0 0 0))
-  )
-  (polyline (pts (xy 16.51 34.29) (xy 45.72 34.29))
     (stroke (width 0) (type default) (color 0 0 0 0))
   )
@@
     (stroke (width 0) (type default) (color 0 0 0 0))
   )
-  (wire (pts (xy 33.02 25.4) (xy 41.91 25.4))
-    (stroke (width 0) (type default) (color 0 0 0 0))
-  )
   (wire (pts (xy 66.04 137.16) (xy 66.04 146.05))
     (stroke (width 0) (type default) (color 0 0 0 0))
@@
     (stroke (width 0) (type default) (color 0 0 0 0))
   )
-  (polyline (pts (xy 45.72 34.29) (xy 45.72 16.51))
-    (stroke (width 0) (type default) (color 0 0 0 0))
-  )
   (wire (pts (xy 190.5 41.91) (xy 209.55 41.91))
     (stroke (width 0) (type default) (color 0 0 0 0))
@@
     (stroke (width 0) (type default) (color 0 0 0 0))
   )
-  (wire (pts (xy 33.02 27.94) (xy 39.37 27.94))
-    (stroke (width 0) (type default) (color 0 0 0 0))
-  )
   (wire (pts (xy 92.71 146.05) (xy 100.33 146.05))
     (stroke (width 0) (type default) (color 0 0 0 0))
@@
     (stroke (width 0) (type default) (color 0 0 0 0))
   )
-  (polyline (pts (xy 16.51 16.51) (xy 45.72 16.51))
-    (stroke (width 0) (type default) (color 0 0 0 0))
-  )
   (wire (pts (xy 222.25 44.45) (xy 226.06 44.45))
     (stroke (width 0) (type default) (color 0 0 0 0))
@@
     (stroke (width 0) (type default) (color 0 0 0 0))
   )
-  (polyline (pts (xy 16.51 16.51) (xy 16.51 34.29))
-    (stroke (width 0) (type default) (color 0 0 0 0))
-  )
   (wire (pts (xy 143.51 31.75) (xy 198.12 31.75))
     (stroke (width 0) (type default) (color 0 0 0 0))
@@
   )
   (label "SDA" (at 171.45 138.43 0)
-    (effects (font (size 1.27 1.27)) (justify left bottom))
-  )
-  (label "Data Output Headers" (at 208.28 93.98 0)
-    (effects (font (size 1.27 1.27)) (justify left bottom))
-  )
-  (label "Power Input Headers" (at 16.51 16.51 0)
     (effects (font (size 1.27 1.27)) (justify left bottom))
   )
@@
     (pin "1")
   )
-  (symbol (lib_id "power:GND") (at 39.37 27.94 0) (unit 1)
-    (in_bom yes) (on_board yes) (fields_autoplaced)
-    (property "Reference" "#PWR02" (id 0) (at 39.37 34.29 0)
-      (effects (font (size 1.27 1.27)) hide)
-    )
-    (property "Value" "GND" (id 1) (at 39.37 33.02 0))
-    (property "Footprint" "" (id 2) (at 39.37 27.94 0)
-      (effects (font (size 1.27 1.27)) hide)
-    )
-    (property "Datasheet" "" (id 3) (at 39.37 27.94 0)
-      (effects (font (size 1.27 1.27)) hide)
-    )
-    (pin "1")
-  )
   (symbol (lib_id "pspice:CAP") (at 115.57 59.69 0) (unit 1)
     (in_bom yes) (on_board yes) (fields_autoplaced)
@@
     )
     (property "Datasheet" "" (id 3) (at 128.27 49.53 0)
-      (effects (font (size 1.27 1.27)) hide)
-    )
-    (pin "1")
-  )
-  (symbol (lib_id "power:+5V") (at 41.91 25.4 0) (unit 1)
-    (in_bom yes) (on_board yes) (fields_autoplaced)
-    (property "Reference" "#PWR03" (id 0) (at 41.91 29.21 0)
-      (effects (font (size 1.27 1.27)) hide)
-    )
-    (property "Value" "+5V" (id 1) (at 41.91 20.32 0))
-    (property "Footprint" "" (id 2) (at 41.91 25.4 0)
-      (effects (font (size 1.27 1.27)) hide)
-    )
-    (property "Datasheet" "" (id 3) (at 41.91 25.4 0)
       (effects (font (size 1.27 1.27)) hide)
     )
@@
     (pin "9")
   )
-  (symbol (lib_id "Connector:Conn_01x02_Male") (at 27.94 25.4 0) (unit 1)
-    (in_bom yes) (on_board yes) (fields_autoplaced)
-    (property "Reference" "J1" (id 0) (at 28.575 20.32 0))
-    (property "Value" "Power Header" (id 1) (at 28.575 22.86 0))
-    (property "Footprint" "Connector_Molex:Molex_KK-396_A-41791-0002_1x02_P3.96mm_Vertical" (id 2) (at 27.94 25.4 0)
-      (effects (font (size 1.27 1.27)) hide)
-    )
-    (property "Datasheet" "~" (id 3) (at 27.94 25.4 0)
-      (effects (font (size 1.27 1.27)) hide)
-    )
-    (pin "1")
-    (pin "2")
-  )
   (symbol (lib_id "Switch:SW_MEC_5G") (at 46.99 175.26 0) (unit 1)
     (in_bom yes) (on_board yes) (fields_autoplaced)
@@
     )
     (pin "1")
+  )
+  (sheet (at 308.61 218.44) (size 304.8 68.58) (fields_autoplaced)
+    (stroke (width 0.1524) (type solid) (color 0 0 0 0))
+    (fill (color 0 0 0 0.0000))
+    (property "Sheet name" "MCU" (id 0) (at 308.61 217.7284 0)
+      (effects (font (size 1.27 1.27)) (justify left bottom))
+    )
+    (property "Sheet file" "MCU.kicad_sch" (id 1) (at 308.61 287.6046 0)
+      (effects (font (size 1.27 1.27)) (justify left top))
+    )
   )
   (sheet (at 307.34 0) (size 307.34 210.82) (fields_autoplaced)
@@
     (path "/" (page "1"))
     (path "/5174c01b-1620-419c-8a1e-138e3ddf685f" (page "2"))
+    (path "/2e8d0db8-fadc-4b32-a04c-e76fcdae81d9" (page "3"))
   )
   (symbol_instances
@@
       (reference "#PWR01") (unit 1) (value "GND") (footprint "")
     )
-    (path "/36f5ab3a-af85-41aa-9b65-b1273c5969dd"
-      (reference "#PWR02") (unit 1) (value "GND") (footprint "")
-    )
-    (path "/a93d2015-8568-4b5a-a1b1-c3cc51cbfecc"
-      (reference "#PWR03") (unit 1) (value "+5V") (footprint "")
-    )
     (path "/53f468a2-a255-4f2f-9e78-d1bee6294b9c"
       (reference "#PWR04") (unit 1) (value "+3.3V") (footprint "")
@@
       (reference "D3") (unit 1) (value "D") (footprint "Diode_SMD:D_0603_1608Metric_Pad1.05x0.95mm_HandSolder")
     )
-    (path "/d2f9a010-444c-47fa-aecb-4924a25b7181"
-      (reference "J1") (unit 1) (value "Power Header") (footprint "Connector_Molex:Molex_KK-396_A-41791-0002_1x02_P3.96mm_Vertical")
-    )
     (path "/227bd997-2057-4fae-b177-81e1242d4fb1"

Commit message: update sensors
Parts:
- Q1: footprint Library:SOT-23_Handsoldering -> Package_TO_SOT_SMD:SOT-23
- U2: footprint Library:SOP-16L-HX711 -> Package_SO:SOP-16_3.9x9.9mm_P1.27mm
Changed lines of the file:
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@@
     (effects (font (size 1.27 1.27)) (justify left bottom))
-  )
-  (global_label "IR-Out" (shape input) (at 185.42 137.16 0) (fields_autoplaced)
-    (effects (font (size 1.27 1.27)) (justify left))
-    (property "Intersheet References" "${INTERSHEET_REFS}" (id 0) (at 194.4855 137.0806 0)
-      (effects (font (size 1.27 1.27)) (justify left) hide)
-    )
   )
   (global_label "A+" (shape input) (at 53.34 64.77 0) (fields_autoplaced)
@@
     )
   )
-  (global_label "IR-In" (shape input) (at 181.61 134.62 0) (fields_autoplaced)
-    (effects (font (size 1.27 1.27)) (justify left))
-    (property "Intersheet References" "${INTERSHEET_REFS}" (id 0) (at 189.2241 134.5406 0)
-      (effects (font (size 1.27 1.27)) (justify left) hide)
-    )
-  )
   (global_label "E-" (shape input) (at 68.58 62.23 0) (fields_autoplaced)
     (effects (font (size 1.27 1.27)) (justify left))
@@
     )
   )
-  (global_label "Flow-Out" (shape input) (at 184.15 109.22 0) (fields_autoplaced)
-    (effects (font (size 1.27 1.27)) (justify left))
-    (property "Intersheet References" "${INTERSHEET_REFS}" (id 0) (at 195.5741 109.1406 0)
-      (effects (font (size 1.27 1.27)) (justify left) hide)
-    )
-  )
   (global_label "A-" (shape input) (at 60.96 67.31 0) (fields_autoplaced)
     (effects (font (size 1.27 1.27)) (justify left))
@@
     )
   )
+  (hierarchical_label "+3.3V" (shape input) (at 66.04 101.6 0)
+    (effects (font (size 1.27 1.27)) (justify left))
+  )
+  (hierarchical_label "Flow-Out" (shape input) (at 184.15 109.22 0)
+    (effects (font (size 1.27 1.27)) (justify left))
+  )
+  (hierarchical_label "+5V" (shape input) (at 226.06 26.67 0)
+    (effects (font (size 1.27 1.27)) (justify left))
+  )
+  (hierarchical_label "IR-Out" (shape input) (at 185.42 137.16 0)
+    (effects (font (size 1.27 1.27)) (justify left))
+  )
+  (hierarchical_label "IR-In" (shape input) (at 181.61 134.62 0)
+    (effects (font (size 1.27 1.27)) (justify left))
+  )
   (symbol (lib_id "power:+3.3V") (at 66.04 128.27 0) (unit 1)
     (in_bom yes) (on_board yes) (fields_autoplaced)
@@
       (effects (font (size 1.27 1.27)) (justify left))
     )
-    (property "Footprint" "Library:SOT-23_Handsoldering" (id 2) (at 212.09 51.435 0)
+    (property "Footprint" "Package_TO_SOT_SMD:SOT-23" (id 2) (at 212.09 51.435 0)
       (effects (font (size 1.27 1.27) italic) (justify left) hide)
     )
@@
     (property "Reference" "U2" (id 0) (at 170.18 34.29 0))
     (property "Value" "HX711" (id 1) (at 170.18 36.83 0))
-    (property "Footprint" "Library:SOP-16L-HX711" (id 2) (at 158.75 80.01 0)
+    (property "Footprint" "Package_SO:SOP-16_3.9x9.9mm_P1.27mm" (id 2) (at 158.75 80.01 0)
       (effects (font (size 1.27 1.27)) (justify left bottom) hide)
     )
@@
       (reference "D3") (unit 1) (value "D") (footprint "Diode_SMD:D_0603_1608Metric_Pad1.05x0.95mm_HandSolder")
     )
+    (path "/5174c01b-1620-419c-8a1e-138e3ddf685f/9d682b23-08a0-467a-8f1b-dbe66aa2c3ca"
+      (reference "J1") (unit 1) (value "Conn_01x02_Male") (footprint "Connector_Molex:Molex_KK-396_A-41791-0002_1x02_P3.96mm_Vertical")
+    )
     (path "/227bd997-2057-4fae-b177-81e1242d4fb1"
       (reference "J2") (unit 1) (value "Scale Header") (footprint "Connector_Molex:Molex_KK-396_A-41791-0004_1x04_P3.96mm_Vertical")
@@
       (reference "J5") (unit 1) (value "Flowmeter Header") (footprint "Connector_Molex:Molex_KK-396_A-41791-0003_1x03_P3.96mm_Vertical")
     )
-    (path "/5174c01b-1620-419c-8a1e-138e3ddf685f/9d682b23-08a0-467a-8f1b-dbe66aa2c3ca"
-      (reference "J?") (unit 1) (value "Conn_01x02_Male") (footprint "Connector_Molex:Molex_KK-396_A-41791-0002_1x02_P3.96mm_Vertical")
-    )
     (path "/5174c01b-1620-419c-8a1e-138e3ddf685f/b501ee6c-bbbf-4380-8cf2-1e0d3418f86a"
       (reference "L1") (unit 1) (value "3.3uH") (footprint "Inductor_SMD:L_Bourns_SRN6045TA")
     )
     (path "/3ff1c051-914a-404b-8a16-68c00deb8b92"
-      (reference "Q1") (unit 1) (value "2N3905") (footprint "Library:SOT-23_Handsoldering")
+      (reference "Q1") (unit 1) (value "2N3905") (footprint "Package_TO_SOT_SMD:SOT-23")
     )
     (path "/61d4db9c-b9dd-4ee1-a274-970452486f2c"
@@
     )
     (path "/d121f0af-1000-4d96-b3b5-dadc0754d7ac"
-      (reference "U2") (unit 1) (value "HX711") (footprint "Library:SOP-16L-HX711")
+      (reference "U2") (unit 1) (value "HX711") (footprint "Package_SO:SOP-16_3.9x9.9mm_P1.27mm")
     )
     (path "/5174c01b-1620-419c-8a1e-138e3ddf685f/e0218f0f-de2b-4da7-8444-7d98f9594ef7"
