File: Circuit Design/power.kicad_sch (KiCad schematic)
At the start: 0 parts

Commit message: Power Sche
Parts:
- added C10, C11, C12, C13, C14, C8, C9: (no value), symbol Device:C
- added J?: Conn_01x02_Male, Connector_Molex:Molex_KK-396_A-41791-0002_1x02_P3.96mm_Vertical, symbol Connector:Conn_01x02_Male
- added L1: (no value), symbol Device:L
- added R11, R12, R13, R14: (no value), symbol Device:R
- added U3: (no value), symbol Regulator_Linear:LM1117-ADJ
- added U4: (no value), symbol Regulator_Switching:TPS562200
Connections:
- new net: C10.1, R11.2, R12.1, U3.1 (ADJ)
- new net: C13.2, R13.2, R14.1, U4.4 (VFB)
- new net: C11.1, L1.1, U4.2 (SW)
- new net: C11.2, U4.6 (VBST)
- new net +12V: C8.1, C9.1, J?.1 (Pin_1), U3.3 (VI), U4.3 (VIN), U4.5 (EN)
- new net +3.3V: C13.1, C14.1, L1.2, R13.1
- new net +5V: C12.1, R11.1, U3.2 (VO)
- new net GND: C10.2, C12.2, C14.2, C8.2, C9.2, J?.2 (Pin_2), R12.2, R14.2, U4.1 (GND)

Commit message: Adding MCU blank sheet and
Parts:
- C10: value (none) -> 56nF; footprint (none) -> Capacitor_SMD:C_0402_1005Metric
- C11: value (none) -> .1uF; footprint (none) -> Capacitor_SMD:C_0805_2012Metric
- C12: value (none) -> 100uF; footprint (none) -> Capacitor_SMD:CP_Elec_6.3x5.8
- C13: value (none) -> 22pF; footprint (none) -> Capacitor_SMD:C_0201_0603Metric
- C14: value (none) -> 44uF; footprint (none) -> Capacitor_SMD:C_0805_2012Metric
- C8: value (none) -> 10uF; footprint (none) -> Capacitor_SMD:CP_Elec_4x5.8
- C9: value (none) -> 22uf; footprint (none) -> Capacitor_SMD:C_0805_2012Metric
- L1: value (none) -> 3.3uH; footprint (none) -> Inductor_SMD:L_Bourns_SRN6045TA
- R11: value (none) -> 330; footprint (none) -> Resistor_SMD:R_0402_1005Metric
- R12: value (none) -> 1k; footprint (none) -> Resistor_SMD:R_0402_1005Metric
- R13: value (none) -> 30.9k; footprint (none) -> Resistor_SMD:R_0201_0603Metric
- R14: value (none) -> 10k; footprint (none) -> Resistor_SMD:R_0201_0603Metric
- U3: value (none) -> LM1117-ADJ; footprint (none) -> Package_TO_SOT_SMD:SOT-223-3_TabPin2
- U4: value (none) -> TPS562207; footprint (none) -> Package_TO_SOT_SMD:SOT-23-6
Changed lines of the file:
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@@
       (effects (font (size 1.27 1.27)) (justify left))
     )
-    (property "Value" "" (id 1) (at 147.32 80.0099 0)
-      (effects (font (size 1.27 1.27)) (justify left))
-    )
-    (property "Footprint" "" (id 2) (at 143.002 78.74 90)
+    (property "Value" "1k" (id 1) (at 147.32 80.0099 0)
+      (effects (font (size 1.27 1.27)) (justify left))
+    )
+    (property "Footprint" "Resistor_SMD:R_0402_1005Metric" (id 2) (at 143.002 78.74 90)
       (effects (font (size 1.27 1.27)) hide)
     )
@@
       (effects (font (size 1.27 1.27)) (justify left))
     )
-    (property "Value" "" (id 1) (at 147.32 66.0399 0)
-      (effects (font (size 1.27 1.27)) (justify left))
-    )
-    (property "Footprint" "" (id 2) (at 143.002 64.77 90)
+    (property "Value" "330" (id 1) (at 147.32 66.0399 0)
+      (effects (font (size 1.27 1.27)) (justify left))
+    )
+    (property "Footprint" "Resistor_SMD:R_0402_1005Metric" (id 2) (at 143.002 64.77 90)
       (effects (font (size 1.27 1.27)) hide)
     )
@@
       (effects (font (size 1.27 1.27)) hide)
     )
-    (property "Value" "" (id 1) (at 198.12 111.76 0))
+    (property "Value" "+3.3V" (id 1) (at 198.12 111.76 0))
     (property "Footprint" "" (id 2) (at 198.12 116.84 0)
       (effects (font (size 1.27 1.27)) hide)
@@
       (effects (font (size 1.27 1.27)) (justify left))
     )
-    (property "Value" "" (id 1) (at 173.99 127 0)
-      (effects (font (size 1.27 1.27)) (justify left))
-    )
-    (property "Footprint" "" (id 2) (at 171.1452 129.54 0)
+    (property "Value" "22pF" (id 1) (at 173.99 127 0)
+      (effects (font (size 1.27 1.27)) (justify left))
+    )
+    (property "Footprint" "Capacitor_SMD:C_0201_0603Metric" (id 2) (at 171.1452 129.54 0)
       (effects (font (size 1.27 1.27)) hide)
     )
@@
       (effects (font (size 1.27 1.27)) (justify left))
     )
-    (property "Value" "" (id 1) (at 156.21 121.9199 0)
-      (effects (font (size 1.27 1.27)) (justify left))
-    )
-    (property "Footprint" "" (id 2) (at 153.3652 124.46 0)
+    (property "Value" ".1uF" (id 1) (at 156.21 121.9199 0)
+      (effects (font (size 1.27 1.27)) (justify left))
+    )
+    (property "Footprint" "Capacitor_SMD:C_0805_2012Metric" (id 2) (at 153.3652 124.46 0)
       (effects (font (size 1.27 1.27)) hide)
     )
@@
       (effects (font (size 1.27 1.27)) (justify left))
     )
-    (property "Value" "" (id 1) (at 115.57 121.9199 0)
-      (effects (font (size 1.27 1.27)) (justify left))
-    )
-    (property "Footprint" "" (id 2) (at 112.7252 124.46 0)
+    (property "Value" "22uf" (id 1) (at 115.57 121.9199 0)
+      (effects (font (size 1.27 1.27)) (justify left))
+    )
+    (property "Footprint" "Capacitor_SMD:C_0805_2012Metric" (id 2) (at 112.7252 124.46 0)
       (effects (font (size 1.27 1.27)) hide)
     )
@@
       (effects (font (size 1.27 1.27)) hide)
     )
-    (property "Value" "" (id 1) (at 85.09 71.12 0))
+    (property "Value" "+12V" (id 1) (at 85.09 71.12 0))
     (property "Footprint" "" (id 2) (at 85.09 76.2 0)
       (effects (font (size 1.27 1.27)) hide)
@@
       (effects (font (size 1.27 1.27)) hide)
     )
-    (property "Value" "" (id 1) (at 180.34 48.26 0))
+    (property "Value" "+5V" (id 1) (at 180.34 48.26 0))
     (property "Footprint" "" (id 2) (at 180.34 53.34 0)
       (effects (font (size 1.27 1.27)) hide)
@@
       (effects (font (size 1.27 1.27)) (justify left))
     )
-    (property "Value" "" (id 1) (at 184.15 138.4299 0)
-      (effects (font (size 1.27 1.27)) (justify left))
-    )
-    (property "Footprint" "" (id 2) (at 179.832 137.16 90)
+    (property "Value" "10k" (id 1) (at 184.15 138.4299 0)
+      (effects (font (size 1.27 1.27)) (justify left))
+    )
+    (property "Footprint" "Resistor_SMD:R_0201_0603Metric" (id 2) (at 179.832 137.16 90)
       (effects (font (size 1.27 1.27)) hide)
     )
@@
       (effects (font (size 1.27 1.27)) (justify left))
     )
-    (property "Value" "" (id 1) (at 171.45 68.5799 0)
-      (effects (font (size 1.27 1.27)) (justify left))
-    )
-    (property "Footprint" "" (id 2) (at 168.6052 71.12 0)
+    (property "Value" "100uF" (id 1) (at 171.45 68.5799 0)
+      (effects (font (size 1.27 1.27)) (justify left))
+    )
+    (property "Footprint" "Capacitor_SMD:CP_Elec_6.3x5.8" (id 2) (at 168.6052 71.12 0)
       (effects (font (size 1.27 1.27)) hide)
     )
@@
     (in_bom yes) (on_board yes) (fields_autoplaced)
     (property "Reference" "L1" (id 0) (at 166.37 110.49 90))
-    (property "Value" "" (id 1) (at 166.37 113.03 90))
-    (property "Footprint" "" (id 2) (at 166.37 116.84 0)
+    (property "Value" "3.3uH" (id 1) (at 166.37 113.03 90))
+    (property "Footprint" "Inductor_SMD:L_Bourns_SRN6045TA" (id 2) (at 166.37 116.84 0)
       (effects (font (size 1.27 1.27)) hide)
     )
@@
       (effects (font (size 1.27 1.27)) hide)
     )
-    (property "Value" "" (id 1) (at 129.54 99.06 0))
+    (property "Value" "GND" (id 1) (at 129.54 99.06 0))
     (property "Footprint" "" (id 2) (at 129.54 93.98 0)
       (effects (font (size 1.27 1.27)) hide)
@@
       (effects (font (size 1.27 1.27)) hide)
     )
-    (property "Value" "" (id 1) (at 130.81 146.05 0))
+    (property "Value" "GND" (id 1) (at 130.81 146.05 0))
     (property "Footprint" "" (id 2) (at 130.81 140.97 0)
       (effects (font (size 1.27 1.27)) hide)
@@
       (effects (font (size 1.27 1.27)) (justify left))
     )
-    (property "Value" "" (id 1) (at 184.15 126.9999 0)
-      (effects (font (size 1.27 1.27)) (justify left))
-    )
-    (property "Footprint" "" (id 2) (at 179.832 125.73 90)
+    (property "Value" "30.9k" (id 1) (at 184.15 126.9999 0)
+      (effects (font (size 1.27 1.27)) (justify left))
+    )
+    (property "Footprint" "Resistor_SMD:R_0201_0603Metric" (id 2) (at 179.832 125.73 90)
       (effects (font (size 1.27 1.27)) hide)
     )
@@
       (effects (font (size 1.27 1.27)) (justify left))
     )
-    (property "Value" "" (id 1) (at 195.58 126.9999 0)
-      (effects (font (size 1.27 1.27)) (justify left))
-    )
-    (property "Footprint" "" (id 2) (at 192.7352 129.54 0)
+    (property "Value" "44uF" (id 1) (at 195.58 126.9999 0)
+      (effects (font (size 1.27 1.27)) (justify left))
+    )
+    (property "Footprint" "Capacitor_SMD:C_0805_2012Metric" (id 2) (at 192.7352 129.54 0)
       (effects (font (size 1.27 1.27)) hide)
     )
@@
       (effects (font (size 1.27 1.27)) (justify left))
     )
-    (property "Value" "" (id 1) (at 115.57 68.5799 0)
-      (effects (font (size 1.27 1.27)) (justify left))
-    )
-    (property "Footprint" "" (id 2) (at 112.7252 71.12 0)
+    (property "Value" "10uF" (id 1) (at 115.57 68.5799 0)
+      (effects (font (size 1.27 1.27)) (justify left))
+    )
+    (property "Footprint" "Capacitor_SMD:CP_Elec_4x5.8" (id 2) (at 112.7252 71.12 0)
       (effects (font (size 1.27 1.27)) hide)
     )
@@
     (in_bom yes) (on_board yes) (fields_autoplaced)
     (property "Reference" "U4" (id 0) (at 133.35 109.22 0))
-    (property "Value" "" (id 1) (at 133.35 111.76 0))
-    (property "Footprint" "" (id 2) (at 134.62 125.73 0)
+    (property "Value" "TPS562207" (id 1) (at 133.35 111.76 0))
+    (property "Footprint" "Package_TO_SOT_SMD:SOT-23-6" (id 2) (at 134.62 125.73 0)
       (effects (font (size 1.27 1.27)) (justify left) hide)
     )
@@
     (in_bom yes) (on_board yes) (fields_autoplaced)
     (property "Reference" "U3" (id 0) (at 121.92 45.72 0))
-    (property "Value" "" (id 1) (at 121.92 48.26 0))
-    (property "Footprint" "" (id 2) (at 121.92 53.34 0)
+    (property "Value" "LM1117-ADJ" (id 1) (at 121.92 48.26 0))
+    (property "Footprint" "Package_TO_SOT_SMD:SOT-223-3_TabPin2" (id 2) (at 121.92 53.34 0)
       (effects (font (size 1.27 1.27)) hide)
     )
@@
       (effects (font (size 1.27 1.27)) (justify left))
     )
-    (property "Value" "" (id 1) (at 125.73 82.5499 0)
-      (effects (font (size 1.27 1.27)) (justify left))
-    )
-    (property "Footprint" "" (id 2) (at 122.8852 85.09 0)
-      (effects (font (size 1.27 1.27)) hide)
-    )
+    (property "Value" "56nF" (id 1) (at 125.73 82.5499 0)
+      (effects (font (size 1.27 1.27)) (justify left))
+    )
+    (property "Footprint" "Capacitor_SMD:C_0402_1005Metric" (id 2) (at 122.8852 85.09 0)
+      (effects (font (size 1.27 1.27)) hide)
+    )

Commit message: update sensors
Parts:
- gave numbers to parts that had none: 1
Changed lines of the file:
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@@
   (symbol (lib_id "Connector:Conn_01x02_Male") (at 88.9 95.25 0) (unit 1)
     (in_bom yes) (on_board yes) (fields_autoplaced)
-    (property "Reference" "J?" (id 0) (at 89.535 90.17 0))
+    (property "Reference" "J1" (id 0) (at 89.535 90.17 0))
     (property "Value" "Conn_01x02_Male" (id 1) (at 89.535 92.71 0))
     (property "Footprint" "Connector_Molex:Molex_KK-396_A-41791-0002_1x02_P3.96mm_Vertical" (id 2) (at 88.9 95.25 0)
