File: Kool Keg Circuit/Kool Keg.kicad_pcb (KiCad board)
At the start: 2 copper layers, 121.6 x 72.7 mm, 75 parts, among them J1 Power, J2 Scale Header, J3 IR, J4 Flow, J5 Prog, J6 Soloenoid, J7 OLED, Q1 2N3905, Q2 2N3906, SW1 SW_MEC_5G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

Commit message: Update PCB
Parts:
- J1: value Power -> Conn_01x02_Male
- J3: value IR -> IR Header
- J4: value Flow -> Flowmeter Header
- J6: value Soloenoid -> Solenoid Conn, 01x02_Male
- J7: value OLED -> Conn_01x02_Female
- moved R17 6.29 mm to (116.0, 87.1), turned to 90 degrees
Connections:
- U4 pad 11: /MCU Subsystem/I2C1_SCL -> /MCU Subsystem/WEIGHT_CLK
- U4 pad 12: /MCU Subsystem/I2C1_SDA -> /MCU Subsystem/WEIGHT_DATA
- U7 pad 11: unconnected-(U7-Pad11) -> /MCU Subsystem/WEIGHT_DATA
- U7 pad 12: unconnected-(U7-Pad12) -> /MCU Subsystem/WEIGHT_CLK
Routing:
- net /MCU Subsystem/WEIGHT_CLK: track 0.00 -> 45.0 mm, vias 0 -> 2
- net /MCU Subsystem/WEIGHT_DATA: track 0.00 -> 43.2 mm, vias 0 -> 2
- net +3.3V: track 29.7 -> 39.6 mm, vias 6 -> 8
- net GND: track 246.1 -> 236.8 mm, vias 11 -> 12
- net /MCU Subsystem/I2C1_SCL: track 65.1 -> 63.5 mm
- net /MCU Subsystem/I2C0_SDA: track 67.2 -> 68.1 mm
- net /MCU Subsystem/I2C1_SDA: vias 1 -> 3

Commit message: PCB update
Parts:
- C6: footprint Capacitor_SMD:C_0603_1608Metric_Pad1.08x0.95mm_HandSolder -> Capacitor_SMD:C_0805_2012Metric_Pad1.18x1.45mm_HandSolder
- D1, D2, D3: footprint Diode_SMD:D_0805_2012Metric_Pad1.15x1.40mm_HandSolder -> Diode_SMD:D_SOD-323_HandSoldering
- moved R18 0.50 mm to (144.5, 79.9)
Routing:
- net /MCU Subsystem/DISP: track 19.4 -> 18.9 mm
