File: Kool Keg Circuit/power.kicad_sch (KiCad schematic)
At the start: 14 parts, among them U1 LM1117-ADJ, U2 TPS562207

Commit message: Consolidating yet again
Changed lines of the file:
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@@
   (junction (at 152.4 105.41) (diameter 0) (color 0 0 0 0)
   )
-  (junction (at 93.98 78.74) (diameter 0) (color 0 0 0 0)
-  )
   (junction (at 152.4 120.65) (diameter 0) (color 0 0 0 0)
   )
+  (junction (at 105.41 35.56) (diameter 0) (color 0 0 0 0)
+  )
+  (junction (at 115.57 76.2) (diameter 0) (color 0 0 0 0)
+  )
+  (junction (at 93.98 105.41) (diameter 0) (color 0 0 0 0)
+  )
+  (junction (at 138.43 35.56) (diameter 0) (color 0 0 0 0)
+  )
+  (junction (at 161.29 35.56) (diameter 0) (color 0 0 0 0)
+  )
+  (junction (at 138.43 76.2) (diameter 0) (color 0 0 0 0)
+  )
+  (junction (at 163.83 120.65) (diameter 0) (color 0 0 0 0)
+  )
+  (junction (at 173.99 105.41) (diameter 0) (color 0 0 0 0)
+  )
   (junction (at 190.5 105.41) (diameter 0) (color 0 0 0 0)
   )
-  (junction (at 105.41 35.56) (diameter 0) (color 0 0 0 0)
-  )
-  (junction (at 115.57 76.2) (diameter 0) (color 0 0 0 0)
-  )
-  (junction (at 93.98 105.41) (diameter 0) (color 0 0 0 0)
-  )
-  (junction (at 138.43 35.56) (diameter 0) (color 0 0 0 0)
-  )
-  (junction (at 161.29 35.56) (diameter 0) (color 0 0 0 0)
-  )
-  (junction (at 138.43 76.2) (diameter 0) (color 0 0 0 0)
-  )
-  (junction (at 163.83 120.65) (diameter 0) (color 0 0 0 0)
-  )
-  (junction (at 173.99 105.41) (diameter 0) (color 0 0 0 0)
-  )
   (junction (at 134.62 105.41) (diameter 0) (color 0 0 0 0)
   )
@@
     (stroke (width 0) (type default) (color 0 0 0 0))
   )
+  (wire (pts (xy 190.5 105.41) (xy 201.93 105.41))
+    (stroke (width 0) (type default) (color 0 0 0 0))
+  )
   (wire (pts (xy 93.98 35.56) (xy 93.98 62.23))
     (stroke (width 0) (type default) (color 0 0 0 0))
@@
     (stroke (width 0) (type default) (color 0 0 0 0))
   )
-  (wire (pts (xy 190.5 105.41) (xy 201.93 105.41))
-    (stroke (width 0) (type default) (color 0 0 0 0))
-  )
   (wire (pts (xy 123.19 35.56) (xy 138.43 35.56))
     (stroke (width 0) (type default) (color 0 0 0 0))
@@
     (stroke (width 0) (type default) (color 0 0 0 0))
   )
-  (wire (pts (xy 93.98 78.74) (xy 93.98 105.41))
+  (wire (pts (xy 93.98 62.23) (xy 93.98 105.41))
     (stroke (width 0) (type default) (color 0 0 0 0))
   )
@@
   )
   (wire (pts (xy 173.99 105.41) (xy 173.99 115.57))
-    (stroke (width 0) (type default) (color 0 0 0 0))
-  )
-  (wire (pts (xy 93.98 62.23) (xy 93.98 78.74))
     (stroke (width 0) (type default) (color 0 0 0 0))
   )
@@
   (hierarchical_label "GND" (shape input) (at 128.27 138.43 0)
     (effects (font (size 1.27 1.27)) (justify left))
+  )
+  (symbol (lib_id "power:PWR_FLAG") (at 190.5 105.41 0) (unit 1)
+    (in_bom yes) (on_board yes) (fields_autoplaced)
+    (property "Reference" "#FLG0104" (id 0) (at 190.5 103.505 0)
+      (effects (font (size 1.27 1.27)) hide)
+    )
+    (property "Value" "PWR_FLAG" (id 1) (at 190.5 100.33 0))
+    (property "Footprint" "" (id 2) (at 190.5 105.41 0)
+      (effects (font (size 1.27 1.27)) hide)
+    )
+    (property "Datasheet" "~" (id 3) (at 190.5 105.41 0)
+      (effects (font (size 1.27 1.27)) hide)
+    )
+    (pin "1")
   )
   (symbol (lib_id "Device:R") (at 138.43 46.99 0) (unit 1)
@@
     (pin "2")
   )
-  (symbol (lib_id "power:PWR_FLAG") (at 190.5 105.41 0) (unit 1)
-    (in_bom yes) (on_board yes) (fields_autoplaced)
-    (property "Reference" "#FLG0102" (id 0) (at 190.5 103.505 0)
-      (effects (font (size 1.27 1.27)) hide)
-    )
-    (property "Value" "PWR_FLAG" (id 1) (at 190.5 100.33 0))
-    (property "Footprint" "" (id 2) (at 190.5 105.41 0)
-      (effects (font (size 1.27 1.27)) hide)
-    )
-    (property "Datasheet" "~" (id 3) (at 190.5 105.41 0)
-      (effects (font (size 1.27 1.27)) hide)
-    )
-    (pin "1")
-  )
   (symbol (lib_id "Device:R") (at 163.83 127 0) (unit 1)
     (in_bom yes) (on_board yes)
@@
       (effects (font (size 1.27 1.27)) hide)
     )
-    (pin "1")
-  )
-  (symbol (lib_id "power:PWR_FLAG") (at 93.98 78.74 90) (unit 1)
-    (in_bom yes) (on_board yes) (fields_autoplaced)
-    (property "Reference" "#FLG0101" (id 0) (at 92.075 78.74 0)
-      (effects (font (size 1.27 1.27)) hide)
-    )
-    (property "Value" "PWR_FLAG" (id 1) (at 90.17 78.7399 90)
-      (effects (font (size 1.27 1.27)) (justify left))
-    )
-    (property "Footprint" "" (id 2) (at 93.98 78.74 0)
-      (effects (font (size 1.27 1.27)) hide)
-    )
-    (property "Datasheet" "~" (id 3) (at 93.98 78.74 0)
-      (effects (font (size 1.27 1.27)) hide)
-    )

Commit message: Update footprints, init layout
Parts:
- C1, C4, C7: footprint Capacitor_SMD:C_0805_2012Metric -> Capacitor_SMD:C_0805_2012Metric_Pad1.18x1.45mm_HandSolder
- C3: footprint Capacitor_SMD:C_0402_1005Metric -> Capacitor_SMD:C_0805_2012Metric_Pad1.18x1.45mm_HandSolder
- C5: footprint Capacitor_SMD:C_0201_0603Metric -> Capacitor_SMD:C_0805_2012Metric_Pad1.18x1.45mm_HandSolder
- R1, R2: footprint Resistor_SMD:R_0402_1005Metric -> Resistor_SMD:R_0805_2012Metric_Pad1.20x1.40mm_HandSolder
- R3, R4: footprint Resistor_SMD:R_0201_0603Metric -> Resistor_SMD:R_0805_2012Metric_Pad1.20x1.40mm_HandSolder
Changed lines of the file:
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@@
       (effects (font (size 1.27 1.27)) (justify left))
     )
-    (property "Footprint" "Resistor_SMD:R_0402_1005Metric" (id 2) (at 136.652 46.99 90)
+    (property "Footprint" "Resistor_SMD:R_0805_2012Metric_Pad1.20x1.40mm_HandSolder" (id 2) (at 136.652 46.99 90)
       (effects (font (size 1.27 1.27)) hide)
     )
@@
       (effects (font (size 1.27 1.27)) (justify left))
     )
-    (property "Footprint" "Resistor_SMD:R_0201_0603Metric" (id 2) (at 162.052 127 90)
+    (property "Footprint" "Resistor_SMD:R_0805_2012Metric_Pad1.20x1.40mm_HandSolder" (id 2) (at 162.052 127 90)
       (effects (font (size 1.27 1.27)) hide)
     )
@@
       (effects (font (size 1.27 1.27)) (justify left))
     )
-    (property "Footprint" "Capacitor_SMD:C_0805_2012Metric" (id 2) (at 135.5852 113.03 0)
+    (property "Footprint" "Capacitor_SMD:C_0805_2012Metric_Pad1.18x1.45mm_HandSolder" (id 2) (at 135.5852 113.03 0)
       (effects (font (size 1.27 1.27)) hide)
     )
@@
       (effects (font (size 1.27 1.27)) (justify left))
     )
-    (property "Footprint" "Capacitor_SMD:C_0805_2012Metric" (id 2) (at 174.9552 123.19 0)
+    (property "Footprint" "Capacitor_SMD:C_0805_2012Metric_Pad1.18x1.45mm_HandSolder" (id 2) (at 174.9552 123.19 0)
       (effects (font (size 1.27 1.27)) hide)
     )
@@
       (effects (font (size 1.27 1.27)) (justify left))
     )
-    (property "Footprint" "Capacitor_SMD:C_0201_0603Metric" (id 2) (at 153.3652 118.11 0)
+    (property "Footprint" "Capacitor_SMD:C_0805_2012Metric_Pad1.18x1.45mm_HandSolder" (id 2) (at 153.3652 118.11 0)
       (effects (font (size 1.27 1.27)) hide)
     )
@@
       (effects (font (size 1.27 1.27)) (justify left))
     )
-    (property "Footprint" "Resistor_SMD:R_0201_0603Metric" (id 2) (at 162.052 114.3 90)
+    (property "Footprint" "Resistor_SMD:R_0805_2012Metric_Pad1.20x1.40mm_HandSolder" (id 2) (at 162.052 114.3 90)
       (effects (font (size 1.27 1.27)) hide)
     )
@@
       (effects (font (size 1.27 1.27)) (justify left))
     )
-    (property "Footprint" "Capacitor_SMD:C_0402_1005Metric" (id 2) (at 116.5352 67.31 0)
+    (property "Footprint" "Capacitor_SMD:C_0805_2012Metric_Pad1.18x1.45mm_HandSolder" (id 2) (at 116.5352 67.31 0)
       (effects (font (size 1.27 1.27)) hide)
     )
@@
       (effects (font (size 1.27 1.27)) (justify left))
     )
-    (property "Footprint" "Resistor_SMD:R_0402_1005Metric" (id 2) (at 136.652 60.96 90)
+    (property "Footprint" "Resistor_SMD:R_0805_2012Metric_Pad1.20x1.40mm_HandSolder" (id 2) (at 136.652 60.96 90)
       (effects (font (size 1.27 1.27)) hide)
     )
@@
       (effects (font (size 1.27 1.27)) (justify left))
     )
-    (property "Footprint" "Capacitor_SMD:C_0805_2012Metric" (id 2) (at 94.9452 120.65 0)
-      (effects (font (size 1.27 1.27)) hide)
-    )
+    (property "Footprint" "Capacitor_SMD:C_0805_2012Metric_Pad1.18x1.45mm_HandSolder" (id 2) (at 94.9452 120.65 0)
+      (effects (font (size 1.27 1.27)) hide)
+    )

Commit message: PCB
Parts:
- added C1: 100nF, Capacitor_SMD:C_0805_2012Metric_Pad1.18x1.45mm_HandSolder, symbol Device:C
- added C4: 10uF, Capacitor_SMD:C_0805_2012Metric_Pad1.18x1.45mm_HandSolder, symbol Device:C
- added C9: 22uF, Capacitor_SMD:C_0805_2012Metric_Pad1.18x1.45mm_HandSolder, symbol Device:C
- C10: renamed from C7; value 44uF -> 22uF
- C3: value 56nF -> 68nF
- C5: renamed from C1; value 22uf -> 10uF
- C6: renamed from C4; footprint Capacitor_SMD:C_0805_2012Metric_Pad1.18x1.45mm_HandSolder -> Capacitor_SMD:C_0603_1608Metric_Pad1.08x0.95mm_HandSolder
- C8: renamed from C5; value 22pF -> 56pF; footprint Capacitor_SMD:C_0805_2012Metric_Pad1.18x1.45mm_HandSolder -> Capacitor_SMD:C_0603_1608Metric_Pad1.08x0.95mm_HandSolder
- U2: footprint Package_TO_SOT_SMD:SOT-23-6 -> Package_TO_SOT_SMD:SOT-563
- renumbered C6 to C7
Connections:
- net +12V: now also U2.1 (VIN), C1.1, C4.1; no longer U2.3 (VIN)
- net +3.3V: now also C9.1
- net GND: now also U2.3 (GND), C1.2, C4.2, C9.2; no longer U2.1 (GND)
- net at C8.2, R3.2, R4.1: now also U2.6 (VFB); no longer U2.4 (VFB)
- net at C6.2: now also U2.4 (VBST); no longer U2.6 (VBST)
Other:
- moved on the sheet: C10, C5, C6, C8, L1, R3, R4, U2

Commit message: PCB update
Parts:
- C6: footprint Capacitor_SMD:C_0603_1608Metric_Pad1.08x0.95mm_HandSolder -> Capacitor_SMD:C_0805_2012Metric_Pad1.18x1.45mm_HandSolder
Changed lines of the file:
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@@
       (effects (font (size 1.27 1.27)) (justify left))
     )
-    (property "Footprint" "Capacitor_SMD:C_0603_1608Metric_Pad1.08x0.95mm_HandSolder" (id 2) (at 155.9052 113.03 0)
+    (property "Footprint" "Capacitor_SMD:C_0805_2012Metric_Pad1.18x1.45mm_HandSolder" (id 2) (at 155.9052 113.03 0)
       (effects (font (size 1.27 1.27)) hide)
     )
