File: Kool Keg Circuit/sensors.kicad_sch (KiCad schematic)
At the start: 29 parts, among them J2 Scale Header, J3 IR Header, J4 Flowmeter Header, Q1 2N3905, SW1 SW_MEC_5G, SW2 SW_MEC_5G, SW3 SW_MEC_5G, U3 74LVC3G14, U4 HX711

Commit message: Update footprints, init layout
Parts:
- C10, C11, C12, C13, C14, C8, C9: footprint Capacitor_SMD:C_0603_1608Metric_Pad1.08x0.95mm_HandSolder -> Capacitor_SMD:C_0805_2012Metric_Pad1.18x1.45mm_HandSolder
- D1, D2, D3: footprint Diode_SMD:D_0603_1608Metric_Pad1.05x0.95mm_HandSolder -> Diode_SMD:D_0805_2012Metric_Pad1.15x1.40mm_HandSolder
- J2, J3: footprint Connector_Molex:Molex_KK-396_A-41791-0004_1x04_P3.96mm_Vertical -> Connector_PinHeader_2.00mm:PinHeader_1x04_P2.00mm_Vertical
- J4: footprint Connector_Molex:Molex_KK-396_A-41791-0003_1x03_P3.96mm_Vertical -> Connector_PinHeader_2.00mm:PinHeader_1x03_P2.00mm_Vertical
- R10, R11, R12, R13, R14, R5, R6, R7, R8, R9: footprint Resistor_SMD:R_0603_1608Metric_Pad0.98x0.95mm_HandSolder -> Resistor_SMD:R_0805_2012Metric_Pad1.20x1.40mm_HandSolder
Changed lines of the file:
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@@
     (property "Reference" "D3" (id 0) (at 86.36 102.87 0))
     (property "Value" "D" (id 1) (at 86.36 105.41 0))
-    (property "Footprint" "Diode_SMD:D_0603_1608Metric_Pad1.05x0.95mm_HandSolder" (id 2) (at 86.36 109.22 0)
+    (property "Footprint" "Diode_SMD:D_0805_2012Metric_Pad1.15x1.40mm_HandSolder" (id 2) (at 86.36 109.22 0)
       (effects (font (size 1.27 1.27)) hide)
     )
@@
       (effects (font (size 1.27 1.27)) (justify left))
     )
-    (property "Footprint" "Resistor_SMD:R_0603_1608Metric_Pad0.98x0.95mm_HandSolder" (id 2) (at 71.882 130.81 90)
+    (property "Footprint" "Resistor_SMD:R_0805_2012Metric_Pad1.20x1.40mm_HandSolder" (id 2) (at 71.882 130.81 90)
       (effects (font (size 1.27 1.27)) hide)
     )
@@
     (property "Reference" "R10" (id 0) (at 86.36 113.03 90))
     (property "Value" "22000" (id 1) (at 86.36 115.57 90))
-    (property "Footprint" "Resistor_SMD:R_0603_1608Metric_Pad0.98x0.95mm_HandSolder" (id 2) (at 86.36 119.888 90)
+    (property "Footprint" "Resistor_SMD:R_0805_2012Metric_Pad1.20x1.40mm_HandSolder" (id 2) (at 86.36 119.888 90)
       (effects (font (size 1.27 1.27)) hide)
     )
@@
       (effects (font (size 1.27 1.27)) (justify left))
     )
-    (property "Footprint" "Resistor_SMD:R_0603_1608Metric_Pad0.98x0.95mm_HandSolder" (id 2) (at 149.352 40.64 90)
+    (property "Footprint" "Resistor_SMD:R_0805_2012Metric_Pad1.20x1.40mm_HandSolder" (id 2) (at 149.352 40.64 90)
       (effects (font (size 1.27 1.27)) hide)
     )
@@
     (property "Reference" "J3" (id 0) (at 219.075 135.89 0))
     (property "Value" "IR Header" (id 1) (at 219.075 138.43 0))
-    (property "Footprint" "Connector_Molex:Molex_KK-396_A-41791-0004_1x04_P3.96mm_Vertical" (id 2) (at 218.44 143.51 0)
+    (property "Footprint" "Connector_PinHeader_2.00mm:PinHeader_1x04_P2.00mm_Vertical" (id 2) (at 218.44 143.51 0)
       (effects (font (size 1.27 1.27)) hide)
     )
@@
     (property "Reference" "C13" (id 0) (at 220.98 67.31 90))
     (property "Value" "0.1uF" (id 1) (at 220.98 69.85 90))
-    (property "Footprint" "Capacitor_SMD:C_0603_1608Metric_Pad1.08x0.95mm_HandSolder" (id 2) (at 223.52 64.77 0)
+    (property "Footprint" "Capacitor_SMD:C_0805_2012Metric_Pad1.18x1.45mm_HandSolder" (id 2) (at 223.52 64.77 0)
       (effects (font (size 1.27 1.27)) hide)
     )
@@
       (effects (font (size 1.27 1.27)) (justify left))
     )
-    (property "Footprint" "Capacitor_SMD:C_0603_1608Metric_Pad1.08x0.95mm_HandSolder" (id 2) (at 217.17 30.48 0)
+    (property "Footprint" "Capacitor_SMD:C_0805_2012Metric_Pad1.18x1.45mm_HandSolder" (id 2) (at 217.17 30.48 0)
       (effects (font (size 1.27 1.27)) hide)
     )
@@
       (effects (font (size 1.27 1.27)) (justify left))
     )
-    (property "Footprint" "Capacitor_SMD:C_0603_1608Metric_Pad1.08x0.95mm_HandSolder" (id 2) (at 100.33 180.34 0)
+    (property "Footprint" "Capacitor_SMD:C_0805_2012Metric_Pad1.18x1.45mm_HandSolder" (id 2) (at 100.33 180.34 0)
       (effects (font (size 1.27 1.27)) hide)
     )
@@
     (property "Reference" "J2" (id 0) (at 52.705 53.34 0))
     (property "Value" "Scale Header" (id 1) (at 52.705 55.88 0))
-    (property "Footprint" "Connector_Molex:Molex_KK-396_A-41791-0004_1x04_P3.96mm_Vertical" (id 2) (at 52.07 60.96 0)
+    (property "Footprint" "Connector_PinHeader_2.00mm:PinHeader_1x04_P2.00mm_Vertical" (id 2) (at 52.07 60.96 0)
       (effects (font (size 1.27 1.27)) hide)
     )
@@
       (effects (font (size 1.27 1.27)) (justify left))
     )
-    (property "Footprint" "Resistor_SMD:R_0603_1608Metric_Pad0.98x0.95mm_HandSolder" (id 2) (at 71.882 158.75 90)
+    (property "Footprint" "Resistor_SMD:R_0805_2012Metric_Pad1.20x1.40mm_HandSolder" (id 2) (at 71.882 158.75 90)
       (effects (font (size 1.27 1.27)) hide)
     )
@@
     (property "Reference" "R9" (id 0) (at 85.09 168.91 90))
     (property "Value" "22000" (id 1) (at 85.09 171.45 90))
-    (property "Footprint" "Resistor_SMD:R_0603_1608Metric_Pad0.98x0.95mm_HandSolder" (id 2) (at 85.09 172.212 90)
+    (property "Footprint" "Resistor_SMD:R_0805_2012Metric_Pad1.20x1.40mm_HandSolder" (id 2) (at 85.09 172.212 90)
       (effects (font (size 1.27 1.27)) hide)
     )
@@
       (effects (font (size 1.27 1.27)) (justify left))
     )
-    (property "Footprint" "Capacitor_SMD:C_0603_1608Metric_Pad1.08x0.95mm_HandSolder" (id 2) (at 100.33 151.13 0)
+    (property "Footprint" "Capacitor_SMD:C_0805_2012Metric_Pad1.18x1.45mm_HandSolder" (id 2) (at 100.33 151.13 0)
       (effects (font (size 1.27 1.27)) hide)
     )
@@
     (property "Reference" "R12" (id 0) (at 115.57 67.31 90))
     (property "Value" "100" (id 1) (at 115.57 69.85 90))
-    (property "Footprint" "Resistor_SMD:R_0603_1608Metric_Pad0.98x0.95mm_HandSolder" (id 2) (at 115.57 66.548 90)
+    (property "Footprint" "Resistor_SMD:R_0805_2012Metric_Pad1.20x1.40mm_HandSolder" (id 2) (at 115.57 66.548 90)
       (effects (font (size 1.27 1.27)) hide)
     )
@@
       (effects (font (size 1.27 1.27)) (justify left))
     )
-    (property "Footprint" "Resistor_SMD:R_0603_1608Metric_Pad0.98x0.95mm_HandSolder" (id 2) (at 71.882 104.14 90)
+    (property "Footprint" "Resistor_SMD:R_0805_2012Metric_Pad1.20x1.40mm_HandSolder" (id 2) (at 71.882 104.14 90)
       (effects (font (size 1.27 1.27)) hide)
     )
@@
     (property "Reference" "C14" (id 0) (at 240.03 34.29 90))
     (property "Value" "10uF" (id 1) (at 240.03 36.83 90))
-    (property "Footprint" "Capacitor_SMD:C_0603_1608Metric_Pad1.08x0.95mm_HandSolder" (id 2) (at 240.03 43.18 0)
+    (property "Footprint" "Capacitor_SMD:C_0805_2012Metric_Pad1.18x1.45mm_HandSolder" (id 2) (at 240.03 43.18 0)
       (effects (font (size 1.27 1.27)) hide)
     )
@@
     (property "Reference" "J4" (id 0) (at 220.345 110.49 0))
     (property "Value" "Flowmeter Header" (id 1) (at 220.345 113.03 0))
-    (property "Footprint" "Connector_Molex:Molex_KK-396_A-41791-0003_1x03_P3.96mm_Vertical" (id 2) (at 219.71 118.11 0)
+    (property "Footprint" "Connector_PinHeader_2.00mm:PinHeader_1x03_P2.00mm_Vertical" (id 2) (at 219.71 118.11 0)
       (effects (font (size 1.27 1.27)) hide)
     )
@@
     (property "Reference" "R13" (id 0) (at 140.97 41.91 90))
     (property "Value" "8.2k" (id 1) (at 140.97 44.45 90))
-    (property "Footprint" "Resistor_SMD:R_0603_1608Metric_Pad0.98x0.95mm_HandSolder" (id 2) (at 140.97 50.038 90)
+    (property "Footprint" "Resistor_SMD:R_0805_2012Metric_Pad1.20x1.40mm_HandSolder" (id 2) (at 140.97 50.038 90)
       (effects (font (size 1.27 1.27)) hide)
     )
@@
     (property "Reference" "D2" (id 0) (at 85.09 157.48 0))
     (property "Value" "D" (id 1) (at 85.09 160.02 0))
-    (property "Footprint" "Diode_SMD:D_0603_1608Metric_Pad1.05x0.95mm_HandSolder" (id 2) (at 85.09 163.83 0)
+    (property "Footprint" "Diode_SMD:D_0805_2012Metric_Pad1.15x1.40mm_HandSolder" (id 2) (at 85.09 163.83 0)
       (effects (font (size 1.27 1.27)) hide)
     )
@@
     (property "Reference" "R8" (id 0) (at 85.09 139.7 90))
     (property "Value" "22000" (id 1) (at 85.09 142.24 90))
-    (property "Footprint" "Resistor_SMD:R_0603_1608Metric_Pad0.98x0.95mm_HandSolder" (id 2) (at 85.09 143.002 90)
+    (property "Footprint" "Resistor_SMD:R_0805_2012Metric_Pad1.20x1.40mm_HandSolder" (id 2) (at 85.09 143.002 90)
       (effects (font (size 1.27 1.27)) hide)
     )
@@
       (effects (font (size 1.27 1.27)) (justify left))
     )
-    (property "Footprint" "Capacitor_SMD:C_0603_1608Metric_Pad1.08x0.95mm_HandSolder" (id 2) (at 100.33 129.54 0)
+    (property "Footprint" "Capacitor_SMD:C_0805_2012Metric_Pad1.18x1.45mm_HandSolder" (id 2) (at 100.33 129.54 0)
       (effects (font (size 1.27 1.27)) hide)
     )
@@
     (property "Reference" "D1" (id 0) (at 85.09 129.54 0))
     (property "Value" "D" (id 1) (at 85.09 132.08 0))
-    (property "Footprint" "Diode_SMD:D_0603_1608Metric_Pad1.05x0.95mm_HandSolder" (id 2) (at 85.09 135.89 0)
+    (property "Footprint" "Diode_SMD:D_0805_2012Metric_Pad1.15x1.40mm_HandSolder" (id 2) (at 85.09 135.89 0)
       (effects (font (size 1.27 1.27)) hide)
     )
@@
     (property "Reference" "R11" (id 0) (at 115.57 46.99 90))
     (property "Value" "100" (id 1) (at 115.57 49.53 90))
-    (property "Footprint" "Resistor_SMD:R_0603_1608Metric_Pad0.98x0.95mm_HandSolder" (id 2) (at 115.57 53.848 90)
+    (property "Footprint" "Resistor_SMD:R_0805_2012Metric_Pad1.20x1.40mm_HandSolder" (id 2) (at 115.57 53.848 90)
       (effects (font (size 1.27 1.27)) hide)
     )
@@
       (effects (font (size 1.27 1.27)) (justify left))
     )
-    (property "Footprint" "Capacitor_SMD:C_0603_1608Metric_Pad1.08x0.95mm_HandSolder" (id 2) (at 123.19 58.42 0)
-      (effects (font (size 1.27 1.27)) hide)
-    )
+    (property "Footprint" "Capacitor_SMD:C_0805_2012Metric_Pad1.18x1.45mm_HandSolder" (id 2) (at 123.19 58.42 0)
+      (effects (font (size 1.27 1.27)) hide)
+    )

Commit message: PCB
Parts:
- SW1, SW2, SW3: footprint Button_Switch_THT:KSA_Tactile_SPST -> Button_Switch_THT:SW_PUSH-12mm; symbol Switch:SW_MEC_5G -> Switch:SW_Push
- renumbered C8 to C11, C9 to C12, C10 to C13, C11 to C14, C12 to C15, C13 to C16, C14 to C17
Connections:
- net Btn1-GPIO: now also U3.5; no longer U3.7
- net Btn2-GPIO: now also U3.7; no longer U3.2
- net Btn3-GPIO: now also U3.2; no longer U3.5
- net GND: no longer SW1.2 (A), SW2.2 (A), SW3.2 (A)
- net IR-In: now also J3.4 (Pin_4); no longer J3.3 (Pin_3)
- net IR-Out: now also J3.3 (Pin_3); no longer J3.4 (Pin_4)
- net at C11.1, D3.1 (K), R10.2: now also U3.3; no longer U3.1
- net at D3.2 (A), R10.1, R5.2: now also SW1.2; no longer SW1.3 (B), SW1.4 (B)
- net at D1.2 (A), R6.2, R8.2: now also SW2.2; no longer SW2.3 (B), SW2.4 (B)
- net at D2.2 (A), R7.2, R9.1: now also SW3.2; no longer SW3.3 (B), SW3.4 (B)
- net at C12.1, D1.1 (K), R8.1: now also U3.1; no longer U3.6
- net at C13.1, D2.1 (K), R9.2: now also U3.6; no longer U3.3

Commit message: PCB update
Parts:
- D1, D2, D3: footprint Diode_SMD:D_0805_2012Metric_Pad1.15x1.40mm_HandSolder -> Diode_SMD:D_SOD-323_HandSoldering
Changed lines of the file:
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@@
     (property "Reference" "D3" (id 0) (at 86.36 102.87 0))
     (property "Value" "D" (id 1) (at 86.36 105.41 0))
-    (property "Footprint" "Diode_SMD:D_0805_2012Metric_Pad1.15x1.40mm_HandSolder" (id 2) (at 86.36 109.22 0)
+    (property "Footprint" "Diode_SMD:D_SOD-323_HandSoldering" (id 2) (at 86.36 109.22 0)
       (effects (font (size 1.27 1.27)) hide)
     )
@@
     (property "Reference" "D2" (id 0) (at 85.09 157.48 0))
     (property "Value" "D" (id 1) (at 85.09 160.02 0))
-    (property "Footprint" "Diode_SMD:D_0805_2012Metric_Pad1.15x1.40mm_HandSolder" (id 2) (at 85.09 163.83 0)
+    (property "Footprint" "Diode_SMD:D_SOD-323_HandSoldering" (id 2) (at 85.09 163.83 0)
       (effects (font (size 1.27 1.27)) hide)
     )
@@
     (property "Reference" "D1" (id 0) (at 85.09 129.54 0))
     (property "Value" "D" (id 1) (at 85.09 132.08 0))
-    (property "Footprint" "Diode_SMD:D_0805_2012Metric_Pad1.15x1.40mm_HandSolder" (id 2) (at 85.09 135.89 0)
-      (effects (font (size 1.27 1.27)) hide)
-    )
+    (property "Footprint" "Diode_SMD:D_SOD-323_HandSoldering" (id 2) (at 85.09 135.89 0)
+      (effects (font (size 1.27 1.27)) hide)
+    )
